File: dac/dac.kicad_pcb (KiCad board)
At the start: 4 copper layers, 50 x 25 mm, 34 parts, among them J1 USB_B, J2 Conn_01x04_Pin, J3 Conn_01x04_Pin, U1 PCM2902, U2 SPX3819M5-L, Y1 12MHz

Commit message: changed U1 name to correct chip PCM2906C
Parts:
- U1: value PCM2902 -> PCM2906C
Changed lines of the file:
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@@
 			)
 		)
-		(property "Value" "PCM2902"
+		(property "Value" "PCM2906C"
 			(at 0 6.25 0)
 			(layer "F.Fab")
@@
 			)
 		)
-		(property "Datasheet" "http://www.ti.com/lit/ds/symlink/pcm2902c.pdf"
+		(property "Datasheet" ""
 			(at 0 0 0)
 			(unlocked yes)
@@
 	)
 	(zone
-		(net 23)
-		(net_name "/VINR")
+		(net 7)
+		(net_name "3V7")
 		(layer "F.Cu")
-		(name "$teardrop_padvia$")
-		(hatch full 0.1)
-		(priority 30007)
-		(attr
-			(teardrop
-				(type padvia)
-			)
-		)
+		(hatch edge 0.5)
+		(priority 2)
 		(connect_pads yes
-			(clearance 0)
+			(clearance 0.2032)
 		)
-		(min_thickness 0.0254)
+		(min_thickness 0.25)
 		(filled_areas_thickness no)
 		(fill yes
@@
 		(polygon
 			(pts
-				(xy 98.426841 90.829475) (xy 98.570525 90.973159) (xy 98.69 91.045) (xy 99.565707 90.819293) (xy 98.69 90.660946)
+				(xy 100.5 88.65) (xy 98.05 88.65) (xy 97.85 87.8) (xy 96.55 87.8) (xy 96.1 88.1) (xy 96.1 88.95)
+				(xy 96.4 89.3) (xy 97.7 89.45) (xy 98.05 89.1) (xy 100.5 89.1)
 			)
 		)
 	)
 	(zone
-		(net 1)
-		(net_name "/VCOM")
+		(net 24)
+		(net_name "/VINL")
 		(layer "F.Cu")
 		(name "$teardrop_padvia$")
 		(hatch full 0.1)
-		(priority 30006)
+		(priority 30005)
 		(attr
 			(teardrop
@@
 		(polygon
 			(pts
-				(xy 99.692 91.5) (xy 99.438 91.5) (xy 99.287836 91.985195) (xy 99.565 92.101) (xy 99.842164 91.985195)
+				(xy 98.443 93.4526) (xy 98.443 93.2494) (xy 98.024229 93.043179) (xy 97.7645 93.351) (xy 98.024229 93.658821)
 			)
 		)
 	)
 	(zone
-		(net 7)
-		(net_name "3V7")
+		(net 18)
+		(net_name "/VOUTR")
 		(layer "F.Cu")
-		(hatch edge 0.5)
-		(priority 2)
+		(name "$teardrop_padvia$")
+		(hatch full 0.1)
+		(priority 30002)
+		(attr
+			(teardrop
+				(type padvia)
+			)
+		)
 		(connect_pads yes
-			(clearance 0.2032)
+			(clearance 0)
 		)
-		(min_thickness 0.25)
+		(min_thickness 0.0254)
 		(filled_areas_thickness no)
 		(fill yes
@@
 		(polygon
 			(pts
-				(xy 100.5 88.65) (xy 98.05 88.65) (xy 97.85 87.8) (xy 96.55 87.8) (xy 96.1 88.1) (xy 96.1 88.95)
-				(xy 96.4 89.3) (xy 97.7 89.45) (xy 98.05 89.1) (xy 100.5 89.1)
+				(xy 106.892 94.084782) (xy 106.638 94.084782) (xy 106.179702 95.419719) (xy 106.965 95.746) (xy 107.750298 95.419719)
 			)
 		)
 	)
 	(zone
-		(net 1)
-		(net_name "/VCOM")
+		(net 8)
+		(net_name "VBUS")
 		(layer "F.Cu")
 		(name "$teardrop_padvia$")
 		(hatch full 0.1)
-		(priority 30008)
+		(priority 30000)
 		(attr
 			(teardrop
@@
 		(polygon
 			(pts
-				(xy 99.438 91.92) (xy 99.692 91.92) (xy 99.79 91.695) (xy 99.565 91.469) (xy 99.34 91.695)
+				(xy 97.645 95.491) (xy 97.645 95.999) (xy 98.495 96.595) (xy 99.346 95.745) (xy 98.495 94.895)
 			)
 		)
 	)
 	(zone
-		(net 20)
-		(net_name "/VOUTL")
+		(net 7)
+		(net_name "3V7")
 		(layer "F.Cu")
-		(name "$teardrop_padvia$")
-		(hatch full 0.1)
-		(priority 30001)
-		(attr
-			(teardrop
-				(type padvia)
-			)
-		)
+		(hatch edge 0.5)
+		(priority 1)
 		(connect_pads yes
-			(clearance 0)
+			(clearance 0.2032)
 		)
-		(min_thickness 0.0254)
+		(min_thickness 0.25)
 		(filled_areas_thickness no)
 		(fill yes
 			(thermal_gap 0.5)
 			(thermal_bridge_width 0.5)
-			(island_removal_mode 1)
-			(island_area_min 10)
 		)
 		(polygon
 			(pts
-				(xy 104.552 94.045) (xy 104.298 94.045) (xy 103.639702 95.419719) (xy 104.425 95.746) (xy 105.210298 95.419719)
+				(xy 90.7976 86.0508) (xy 90.7976 84.7008) (xy 91.2 84.4) (xy 94.6 84.4) (xy 98.15 87.5) (xy 98.15 89)
+				(xy 97.7 89.45) (xy 96.15 89.45) (xy 94.95 88.7) (xy 90.855 88.65) (xy 90.8812 88.0364)
 			)
 		)
 	)
 	(zone
-		(net 20)
-		(net_name "/VOUTL")
+		(net 1)
+		(net_name "/VCOM")
 		(layer "F.Cu")
 		(name "$teardrop_padvia$")
 		(hatch full 0.1)
-		(priority 30003)
+		(priority 30006)
 		(attr
 			(teardrop
@@
 		(polygon
 			(pts
-				(xy 105.665 90.693) (xy 105.665 90.947) (xy 105.89 91.045) (xy 106.766 90.82) (xy 105.89 90.595)
+				(xy 99.692 91.5) (xy 99.438 91.5) (xy 99.287836 91.985195) (xy 99.565 92.101) (xy 99.842164 91.985195)
 			)
 		)
 	)
 	(zone
-		(net 8)
-		(net_name "VBUS")
+		(net 23)
+		(net_name "/VINR")
 		(layer "F.Cu")
 		(name "$teardrop_padvia$")
 		(hatch full 0.1)
-		(priority 30000)
+		(priority 30007)
 		(attr
 			(teardrop
@@
 		(polygon
 			(pts
-				(xy 97.645 95.491) (xy 97.645 95.999) (xy 98.495 96.595) (xy 99.346 95.745) (xy 98.495 94.895)
+				(xy 98.426841 90.829475) (xy 98.570525 90.973159) (xy 98.69 91.045) (xy 99.565707 90.819293) (xy 98.69 90.660946)
 			)
 		)
 	)
 	(zone
-		(net 24)
-		(net_name "/VINL")
+		(net 20)
+		(net_name "/VOUTL")
 		(layer "F.Cu")
 		(name "$teardrop_padvia$")
 		(hatch full 0.1)
-		(priority 30005)
+		(priority 30003)
 		(attr
 			(teardrop
@@
 		(polygon
 			(pts
-				(xy 98.443 93.4526) (xy 98.443 93.2494) (xy 98.024229 93.043179) (xy 97.7645 93.351) (xy 98.024229 93.658821)
+				(xy 105.665 90.693) (xy 105.665 90.947) (xy 105.89 91.045) (xy 106.766 90.82) (xy 105.89 90.595)
 			)
 		)
 	)
 	(zone
-		(net 7)
-		(net_name "3V7")
+		(net 2)
+		(net_name "GND")
 		(layer "F.Cu")
 		(hatch edge 0.5)
-		(priority 1)
 		(connect_pads yes
 			(clearance 0.2032)
@@
 		(polygon
 			(pts
-				(xy 90.7976 86.0508) (xy 90.7976 84.7008) (xy 91.2 84.4) (xy 94.6 84.4) (xy 98.15 87.5) (xy 98.15 89)
-				(xy 97.7 89.45) (xy 96.15 89.45) (xy 94.95 88.7) (xy 90.855 88.65) (xy 90.8812 88.0364)
+				(xy 100.4 89.8) (xy 100.4 89.2) (xy 98.6 89.2) (xy 97.8 89.8) (xy 96.7 89.8) (xy 96.2 90) (xy 96.2 91.3)
+				(xy 96.7 91.5) (xy 97.6 91.5) (xy 98 91.2) (xy 98 90.3) (xy 98.6 89.8)
 			)
 		)
 	)
 	(zone
-		(net 24)
-		(net_name "/VINL")
+		(net 20)
+		(net_name "/VOUTL")
 		(layer "F.Cu")
 		(name "$teardrop_padvia$")
 		(hatch full 0.1)
-		(priority 30004)
+		(priority 30001)
 		(attr
 			(teardrop
@@
 		(polygon
 			(pts
-				(xy 100.586773 90.257256) (xy 100.730456 90.113573) (xy 100.44 89.957169) (xy 99.564293 90.169293)
-				(xy 100.44 90.395)
+				(xy 104.552 94.045) (xy 104.298 94.045) (xy 103.639702 95.419719) (xy 104.425 95.746) (xy 105.210298 95.419719)
 			)
 		)
@@
 	)
 	(zone
-		(net 18)
-		(net_name "/VOUTR")
+		(net 6)
+		(net_name "VDDI")
 		(layer "F.Cu")
-		(name "$teardrop_padvia$")
-		(hatch full 0.1)
-		(priority 30002)
-		(attr
-			(teardrop
-				(type padvia)
-			)
-		)
+		(hatch edge 0.5)
+		(priority 4)
 		(connect_pads yes
-			(clearance 0)
+			(clearance 0.2032)
 		)
-		(min_thickness 0.0254)
+		(min_thickness 0.25)
 		(filled_areas_thickness no)
 		(fill yes
@@
 		(polygon
 			(pts
-				(xy 106.892 94.084782) (xy 106.638 94.084782) (xy 106.179702 95.419719) (xy 106.965 95.746) (xy 107.750298 95.419719)
+				(xy 98.7044 88.4428) (xy 100.4316 88.4428) (xy 100.44 87.345) (xy 98.6028 87.3252)
 			)
 		)
 	)
 	(zone
-		(net 2)
-		(net_name "GND")
+		(net 24)
+		(net_name "/VINL")
 		(layer "F.Cu")
-		(hatch edge 0.5)
+		(name "$teardrop_padvia$")
+		(hatch full 0.1)
+		(priority 30004)
+		(attr
+			(teardrop
+				(type padvia)
+			)
+		)
 		(connect_pads yes
-			(clearance 0.2032)
+			(clearance 0)
 		)
-		(min_thickness 0.25)
+		(min_thickness 0.0254)
 		(filled_areas_thickness no)
 		(fill yes
 			(thermal_gap 0.5)
 			(thermal_bridge_width 0.5)
+			(island_removal_mode 1)
+			(island_area_min 10)
 		)
 		(polygon
 			(pts
-				(xy 100.4 89.8) (xy 100.4 89.2) (xy 98.6 89.2) (xy 97.8 89.8) (xy 96.7 89.8) (xy 96.2 90) (xy 96.2 91.3)
-				(xy 96.7 91.5) (xy 97.6 91.5) (xy 98 91.2) (xy 98 90.3) (xy 98.6 89.8)
+				(xy 100.586773 90.257256) (xy 100.730456 90.113573) (xy 100.44 89.957169) (xy 99.564293 90.169293)
+				(xy 100.44 90.395)
 			)
 		)
 	)
 	(zone
-		(net 6)
-		(net_name "VDDI")
+		(net 1)
+		(net_name "/VCOM")
 		(layer "F.Cu")
-		(hatch edge 0.5)
-		(priority 4)
+		(name "$teardrop_padvia$")
+		(hatch full 0.1)
+		(priority 30008)
+		(attr
+			(teardrop
+				(type padvia)
+			)
+		)
 		(connect_pads yes
-			(clearance 0.2032)
+			(clearance 0)
 		)
-		(min_thickness 0.25)
+		(min_thickness 0.0254)
 		(filled_areas_thickness no)
 		(fill yes
@@
 		(polygon
 			(pts
-				(xy 98.7044 88.4428) (xy 100.4316 88.4428) (xy 100.44 87.345) (xy 98.6028 87.3252)
+				(xy 99.438 91.92) (xy 99.692 91.92) (xy 99.79 91.695) (xy 99.565 91.469) (xy 99.34 91.695)
 			)
 		)
@@
 		(name "$teardrop_padvia$")
 		(hatch full 0.1)
-		(priority 30000)
+		(priority 30001)
 		(attr
 			(teardrop
@@
 		(polygon
 			(pts
-				(xy 99.311 91.7925) (xy 99.819 91.7925) (xy 100.137217 91.165559) (xy 99.536 90.6165) (xy 98.962315 91.183956)
+				(xy 99.819 91.5) (xy 99.311 91.5) (xy 99.265 92.1) (xy 99.565 92.101) (xy 99.865 92.1)
 			)
 		)
@@
 		(name "$teardrop_padvia$")
 		(hatch full 0.1)
-		(priority 30001)
+		(priority 30000)
 		(attr
 			(teardrop
@@
 		(polygon
 			(pts
-				(xy 99.819 91.5) (xy 99.311 91.5) (xy 99.265 92.1) (xy 99.565 92.101) (xy 99.865 92.1)
+				(xy 99.311 91.7925) (xy 99.819 91.7925) (xy 100.137217 91.165559) (xy 99.536 90.6165) (xy 98.962315 91.183956)
 			)
 		)
